File: Powerboard/3v3_Stepdown.kicad_sch (KiCad schematic)
At the start: 16 parts, among them U1 MP2338GTL-Z

Commit message: fixed sch
Parts:
- C1, C2: value C -> 10uF; footprint (none) -> Capacitor_SMD:C_1206_3216Metric
- C3, C5: value C -> 0.1uF; footprint (none) -> Capacitor_SMD:C_0603_1608Metric
- C4: value C -> 22nF; footprint (none) -> Capacitor_SMD:C_0603_1608Metric
- C6, C7: value C -> 22uF; footprint (none) -> Capacitor_SMD:C_1206_3216Metric
- C8: value C -> 470pF; footprint (none) -> Capacitor_SMD:C_0603_1608Metric
- L1: value L -> 6.8uH; footprint (none) -> Inductor_SMD:L_Bourns_SRP7028A_7.3x6.6mm
- R1: value R -> 191k; footprint (none) -> Resistor_SMD:R_0603_1608Metric
- R2: value R -> 49.9k; footprint (none) -> Resistor_SMD:R_0603_1608Metric
- R3: value R -> 100k; footprint (none) -> Resistor_SMD:R_0603_1608Metric
- R4: value R -> 10k; footprint (none) -> Resistor_SMD:R_0603_1608Metric
- R5: value R -> 9.09k; footprint (none) -> Resistor_SMD:R_0603_1608Metric
- R6: value R -> 51k; footprint (none) -> Resistor_SMD:R_0603_1608Metric
- U1: footprint SOT583_MP2338_MNP -> MP2338GTL:SOT583_MP2338_MNP
Other:
- moved on the sheet: C1, C2, C3, C6, C8, R1, R2
