File: Powerboard/5vStep.kicad_sch (KiCad schematic)
At the start: 15 parts, among them U3 MP2338GTL-Z

Commit message: fixed sch
Parts:
- C11, C20: value C -> 22uF; footprint (none) -> Capacitor_SMD:C_1206_3216Metric
- C17, C19: value C -> 0.1uF; footprint (none) -> Capacitor_SMD:C_0603_1608Metric
- C18: value C -> 22nF; footprint (none) -> Capacitor_SMD:C_0603_1608Metric
- C21: value C -> 22uF; footprint (none) -> Capacitor_SMD:C_0603_1608Metric
- C22: value C -> 300pF; footprint (none) -> Capacitor_SMD:C_0603_1608Metric
- L3: value L -> 6.8uH; footprint (none) -> Inductor_SMD:L_Bourns_SRP7028A_7.3x6.6mm
- R13: value R -> 191k; footprint (none) -> Resistor_SMD:R_0603_1608Metric
- R14: value R -> 49.9k; footprint (none) -> Resistor_SMD:R_0603_1608Metric
- R15, R16, R17: value R -> 10k; footprint (none) -> Resistor_SMD:R_0603_1608Metric
- R18: value R -> 90.9k; footprint (none) -> Resistor_SMD:R_0603_1608Metric
- U3: footprint SOT583_MP2338_MNP -> MP2338GTL:SOT583_MP2338_MNP
Other:
- moved on the sheet: C11, C21, R13, R14
