File: Powerboard/Encoder_data.kicad_sch (KiCad schematic)
At the start: 0 parts

Commit message: Finished the board
Parts:
- added U7, U8: SN74LVC245AN, N20, symbol SN74LVC245AN:SN74LVC245AN
Connections:
- new net EA1_3v3: U7.2 (A1)
- new net EA1_5v: U7.18 (B1)
- new net EA2_3v3: U7.4 (A3)
- new net EA2_5v: U7.16 (B3)
- new net EA3_3v3: U7.6 (A5)
- new net EA3_5v: U7.14 (B5)
- new net EA4_3v3: U7.8 (A7)
- new net EA4_5v: U7.12 (B7)
- new net EA5_3v3: U8.2 (A1)
- new net EA5_5v: U8.18 (B1)
- new net EA6_3v3: U8.4 (A3)
- new net EA6_5v: U8.16 (B3)
- new net EB1_3v3: U7.3 (A2)
- new net EB1_5v: U7.17 (B2)
- new net EB2_3v3: U7.5 (A4)
- new net EB2_5v: U7.15 (B4)
- new net EB3_3v3: U7.7 (A6)
- new net EB3_5v: U7.13 (B6)
- new net EB4_3v3: U7.9 (A8)
- new net EB4_5v: U7.11 (B8)
- new net EB5_3v3: U8.3 (A2)
- new net EB5_5v: U8.17 (B2)
- new net EB6_3v3: U8.5 (A4)
- new net EB6_5v: U8.15 (B4)
- new net GND: U7.1 (DIR), U7.10 (GND), U7.19 (*OE), U8.1 (DIR), U8.10 (GND), U8.19 (*OE)
- new net Vout_3v3: U7.20 (VCC), U8.20 (VCC)

Commit message: fixed sch
Parts:
- U7, U8: footprint N20 -> SN74LVC245AN:N20
Connections:
- no-connect marks 0 -> 8
