File: Powerboard/Encoder_data.kicad_sch (KiCad schematic)
At the start: 2 parts, among them U7 SN74LVC245AN, U8 SN74LVC245AN

Commit message: Updated
Parts:
- renumbered U7 to U3, U8 to U4
Changed lines of the file:
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@@
 		(dnp no)
 		(fields_autoplaced yes)
-		(property "Reference" "U7"
+		(property "Reference" "U3"
 			(at 133.35 41.91 0)
 			(show_name no)
@@
 			(project "Powerboard"
 				(path "/07aca59a-bf87-409f-a974-db5a163ccf8c/b0384a87-201b-4948-b16f-22c202c766d2"
-					(reference "U7")
+					(reference "U3")
 					(unit 1)
 				)
@@
 		(dnp no)
 		(fields_autoplaced yes)
-		(property "Reference" "#FLG02"
+		(property "Reference" "#FLG03"
 			(at 165.1 50.165 0)
 			(hide yes)
@@
 			(project "Powerboard"
 				(path "/07aca59a-bf87-409f-a974-db5a163ccf8c/b0384a87-201b-4948-b16f-22c202c766d2"
-					(reference "#FLG02")
+					(reference "#FLG03")
 					(unit 1)
 				)
@@
 		(dnp no)
 		(fields_autoplaced yes)
-		(property "Reference" "U8"
+		(property "Reference" "U4"
 			(at 133.35 86.36 0)
 			(show_name no)
@@
 			(project "Powerboard"
 				(path "/07aca59a-bf87-409f-a974-db5a163ccf8c/b0384a87-201b-4948-b16f-22c202c766d2"
-					(reference "U8")
+					(reference "U4")
 					(unit 1)
 				)
@@
 		(dnp no)
 		(fields_autoplaced yes)
-		(property "Reference" "#FLG01"
+		(property "Reference" "#FLG02"
 			(at 95.885 77.47 0)
 			(hide yes)
@@
 			(project "Powerboard"
 				(path "/07aca59a-bf87-409f-a974-db5a163ccf8c/b0384a87-201b-4948-b16f-22c202c766d2"
-					(reference "#FLG01")
+					(reference "#FLG02")
 					(unit 1)
 				)
@@
 		(dnp no)
 		(fields_autoplaced yes)
-		(property "Reference" "#PWR025"
+		(property "Reference" "#PWR019"
 			(at 96.52 135.89 0)
 			(hide yes)
@@
 			(project "Powerboard"
 				(path "/07aca59a-bf87-409f-a974-db5a163ccf8c/b0384a87-201b-4948-b16f-22c202c766d2"
-					(reference "#PWR025")
+					(reference "#PWR019")
 					(unit 1)
 				)
@@
 		(dnp no)
 		(fields_autoplaced yes)
-		(property "Reference" "#PWR026"
+		(property "Reference" "#PWR020"
 			(at 97.79 86.36 0)
 			(hide yes)
@@
 			(project "Powerboard"
 				(path "/07aca59a-bf87-409f-a974-db5a163ccf8c/b0384a87-201b-4948-b16f-22c202c766d2"
-					(reference "#PWR026")
+					(reference "#PWR020")
 					(unit 1)
 				)

Commit message: update
Parts:
- removed U3, U4: SN74LVC245AN, SN74LVC245AN:N20, symbol SN74LVC245AN:SN74LVC245AN
- added U3, U4: SN74LVC245ADW, SN74LVC245ADW:DW20, symbol SN74LVC245ADW:SN74LVC245ADW
Connections:
- net EA1_3v3: now also U3.9 (A8)
- net EA1_5v: now also U3.11 (B8)
- net EA2_3v3: now also U3.7 (A6)
- net EA2_5v: now also U3.13 (B6)
- net EA3_3v3: now also U3.5 (A4)
- net EA3_5v: now also U3.15 (B4)
- net EA4_3v3: now also U3.3 (A2)
- net EA4_5v: now also U3.17 (B2)
- net EA5_3v3: now also U4.5 (A4)
- net EA5_5v: now also U4.15 (B4)
- net EA6_3v3: now also U4.3 (A2)
- net EA6_5v: now also U4.17 (B2)
- net EB1_3v3: now also U3.8 (A7)
- net EB1_5v: now also U3.12 (B7)
- net EB2_3v3: now also U3.6 (A5)
- net EB2_5v: now also U3.14 (B5)
- net EB3_3v3: now also U3.4 (A3)
- net EB3_5v: now also U3.16 (B3)
- net EB4_3v3: now also U3.2 (A1)
- net EB4_5v: now also U3.18 (B1)
- net EB5_3v3: now also U4.4 (A3)
- net EB5_5v: now also U4.16 (B3)
- net EB6_3v3: now also U4.2 (A1)
- net EB6_5v: now also U4.18 (B1)
- net GND: now also U3.1 (DIR), U3.10 (GND), U3.19 (*OE), U4.1 (DIR), U4.10 (GND), U4.19 (*OE)
- net Vout_3v3: now also U3.20 (VCC), U4.20 (VCC)

Commit message: Rev1.1 Done
Finished the board ran DRC all clear
Other:
- company: (none) -> Visionbyte Labs
- title: (none) -> Arm Powerboard
Changed lines of the file:
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@@
 	(generator_version "10.0")
 	(paper "A4")
+	(title_block
+		(title "Arm Powerboard")
+		(date "2026-08-09")
+		(rev "1.1")
+		(company "Visionbyte Labs")
+	)
 	(junction
 		(at 165.1 52.07)
