File: Powerboard/Motor_Driver.kicad_sch (KiCad schematic)
At the start: 4 parts, among them U2 SN74HCT245N, U4 SN74HCT245N

Commit message: Finished the board
Parts:
- renumbered C10 to C12, C9 to C13, U2 to U5, U4 to U6
Changed lines of the file:
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@@
 		(dnp no)
 		(fields_autoplaced yes)
-		(property "Reference" "U2"
+		(property "Reference" "U5"
 			(at 146.05 30.48 0)
 			(show_name no)
@@
 		(instances
 			(project "Powerboard"
-				(path "/07aca59a-bf87-409f-a974-db5a163ccf8c/671dbe42-136f-4e16-893b-56b15122f6a7"
-					(reference "U2")
+				(path "/07aca59a-bf87-409f-a974-db5a163ccf8c/c97f42c2-abf8-4b30-857d-14b47bb2334c"
+					(reference "U5")
 					(unit 1)
 				)
@@
 		(dnp no)
 		(fields_autoplaced yes)
-		(property "Reference" "#PWR015"
+		(property "Reference" "#PWR016"
 			(at 95.25 77.47 0)
 			(hide yes)
@@
 		(instances
 			(project "Powerboard"
-				(path "/07aca59a-bf87-409f-a974-db5a163ccf8c/671dbe42-136f-4e16-893b-56b15122f6a7"
-					(reference "#PWR015")
+				(path "/07aca59a-bf87-409f-a974-db5a163ccf8c/c97f42c2-abf8-4b30-857d-14b47bb2334c"
+					(reference "#PWR016")
 					(unit 1)
 				)
@@
 		(dnp no)
 		(fields_autoplaced yes)
-		(property "Reference" "C9"
+		(property "Reference" "C13"
 			(at 99.06 113.0299 0)
 			(show_name no)
@@
 		(instances
 			(project "Powerboard"
-				(path "/07aca59a-bf87-409f-a974-db5a163ccf8c/671dbe42-136f-4e16-893b-56b15122f6a7"
-					(reference "C9")
+				(path "/07aca59a-bf87-409f-a974-db5a163ccf8c/c97f42c2-abf8-4b30-857d-14b47bb2334c"
+					(reference "C13")
 					(unit 1)
 				)
@@
 		(dnp no)
 		(fields_autoplaced yes)
-		(property "Reference" "#PWR013"
+		(property "Reference" "#PWR014"
 			(at 95.25 144.78 0)
 			(hide yes)
@@
 		(instances
 			(project "Powerboard"
-				(path "/07aca59a-bf87-409f-a974-db5a163ccf8c/671dbe42-136f-4e16-893b-56b15122f6a7"
-					(reference "#PWR013")
+				(path "/07aca59a-bf87-409f-a974-db5a163ccf8c/c97f42c2-abf8-4b30-857d-14b47bb2334c"
+					(reference "#PWR014")
 					(unit 1)
 				)
@@
 		(dnp no)
 		(fields_autoplaced yes)
-		(property "Reference" "U4"
+		(property "Reference" "U6"
 			(at 148.59 97.79 0)
 			(show_name no)
@@
 		(instances
 			(project "Powerboard"
-				(path "/07aca59a-bf87-409f-a974-db5a163ccf8c/671dbe42-136f-4e16-893b-56b15122f6a7"
-					(reference "U4")
+				(path "/07aca59a-bf87-409f-a974-db5a163ccf8c/c97f42c2-abf8-4b30-857d-14b47bb2334c"
+					(reference "U6")
 					(unit 1)
 				)
@@
 		(dnp no)
 		(fields_autoplaced yes)
-		(property "Reference" "#PWR011"
+		(property "Reference" "#PWR027"
 			(at 180.34 43.18 0)
 			(hide yes)
@@
 		(instances
 			(project "Powerboard"
-				(path "/07aca59a-bf87-409f-a974-db5a163ccf8c/671dbe42-136f-4e16-893b-56b15122f6a7"
-					(reference "#PWR011")
+				(path "/07aca59a-bf87-409f-a974-db5a163ccf8c/c97f42c2-abf8-4b30-857d-14b47bb2334c"
+					(reference "#PWR027")
 					(unit 1)
 				)
@@
 		(dnp no)
 		(fields_autoplaced yes)
-		(property "Reference" "#PWR010"
+		(property "Reference" "#PWR028"
 			(at 182.88 110.49 0)
 			(hide yes)
@@
 		(instances
 			(project "Powerboard"
-				(path "/07aca59a-bf87-409f-a974-db5a163ccf8c/671dbe42-136f-4e16-893b-56b15122f6a7"
-					(reference "#PWR010")
+				(path "/07aca59a-bf87-409f-a974-db5a163ccf8c/c97f42c2-abf8-4b30-857d-14b47bb2334c"
+					(reference "#PWR028")
 					(unit 1)
 				)
@@
 		(dnp no)
 		(fields_autoplaced yes)
-		(property "Reference" "C10"
+		(property "Reference" "C12"
 			(at 99.06 46.9899 0)
 			(show_name no)
@@
 		(instances
 			(project "Powerboard"
-				(path "/07aca59a-bf87-409f-a974-db5a163ccf8c/671dbe42-136f-4e16-893b-56b15122f6a7"
-					(reference "C10")
-					(unit 1)
-				)
+				(path "/07aca59a-bf87-409f-a974-db5a163ccf8c/c97f42c2-abf8-4b30-857d-14b47bb2334c"
+					(reference "C12")
+					(unit 1)
+				)

Commit message: fixed sch
Parts:
- C12, C13: footprint (none) -> Capacitor_SMD:C_0603_1608Metric
- U5, U6: footprint N20 -> SN74HCT245N:N20
Connections:
- no-connect marks 0 -> 8
Changed lines of the file:
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@@
 		(color 0 0 0 0)
 	)
+	(junction
+		(at 95.25 38.1)
+		(diameter 0)
+		(color 0 0 0 0)
+	)
+	(no_connect
+		(at 176.53 125.73)
+	)
+	(no_connect
+		(at 120.65 120.65)
+	)
+	(no_connect
+		(at 120.65 125.73)
+	)
+	(no_connect
+		(at 120.65 128.27)
+	)
+	(no_connect
+		(at 176.53 130.81)
+	)
+	(no_connect
+		(at 176.53 123.19)
+	)
+	(no_connect
+		(at 176.53 128.27)
+	)
+	(no_connect
+		(at 120.65 123.19)
+	)
 	(wire
 		(pts
@@
 	(wire
 		(pts
-			(xy 95.25 33.02) (xy 95.25 40.64)
+			(xy 95.25 33.02) (xy 95.25 38.1)
 		)
 		(stroke
@@
 	(wire
 		(pts
-			(xy 95.25 138.43) (xy 95.25 130.81)
+			(xy 95.25 130.81) (xy 95.25 138.43)
 		)
 		(stroke
@@
 	(wire
 		(pts
+			(xy 179.07 100.33) (xy 179.07 107.95)
+		)
+		(stroke
+			(width 0)
+			(type default)
+		)
+	)
+	(wire
+		(pts
+			(xy 95.25 130.81) (xy 120.65 130.81)
+		)
+		(stroke
+			(width 0)
+			(type default)
+		)
+	)
+	(wire
+		(pts
 			(xy 95.25 63.5) (xy 95.25 71.12)
 		)
@@
 	(wire
 		(pts
-			(xy 179.07 100.33) (xy 179.07 107.95)
-		)
-		(stroke
-			(width 0)
-			(type default)
-		)
-	)
-	(wire
-		(pts
-			(xy 95.25 130.81) (xy 120.65 130.81)
-		)
-		(stroke
-			(width 0)
-			(type default)
-		)
-	)
-	(wire
-		(pts
 			(xy 95.25 40.64) (xy 95.25 44.45)
+		)
+		(stroke
+			(width 0)
+			(type default)
+		)
+	)
+	(wire
+		(pts
+			(xy 95.25 38.1) (xy 95.25 40.64)
 		)
 		(stroke
@@
 			)
 		)
-		(property "Footprint" "N20"
+		(property "Footprint" "SN74HCT245N:N20"
 			(at 118.11 40.64 0)
 			(hide yes)
@@
 		)
 		(property "Description" ""
+			(at 118.11 40.64 0)
+			(hide yes)
+			(show_name no)
+			(do_not_autoplace no)
+			(effects
+				(font
+					(size 1.27 1.27)
+				)
+			)
+		)
+		(property "Untitled Field" ""
 			(at 118.11 40.64 0)
 			(hide yes)
@@
 			)
 		)
-		(property "Footprint" ""
+		(property "Footprint" "Capacitor_SMD:C_0603_1608Metric"
 			(at 96.2152 118.11 0)
 			(hide yes)
@@
 	)
 	(symbol
+		(lib_id "power:PWR_FLAG")
+		(at 95.25 38.1 90)
+		(unit 1)
+		(body_style 1)
+		(exclude_from_sim no)
+		(in_bom yes)
+		(on_board yes)
+		(in_pos_files yes)
+		(dnp no)
+		(fields_autoplaced yes)
+		(property "Reference" "#FLG03"
+			(at 93.345 38.1 0)
+			(hide yes)
+			(show_name no)
+			(do_not_autoplace no)
+			(effects
+				(font
+					(size 1.27 1.27)
+				)
+			)
+		)
+		(property "Value" "PWR_FLAG"
+			(at 91.44 38.0999 90)
+			(show_name no)
+			(do_not_autoplace no)
+			(effects
+				(font
+					(size 1.27 1.27)
+				)
+				(justify left)
+			)
+		)
+		(property "Footprint" ""
+			(at 95.25 38.1 0)
+			(hide yes)
+			(show_name no)
+			(do_not_autoplace no)
+			(effects
+				(font
+					(size 1.27 1.27)
+				)
+			)
+		)
+		(property "Datasheet" ""
+			(at 95.25 38.1 0)
+			(hide yes)
+			(show_name no)
+			(do_not_autoplace no)
+			(effects
+				(font
+					(size 1.27 1.27)
+				)
+			)
+		)
+		(property "Description" "Special symbol for telling ERC where power comes from"
+			(at 95.25 38.1 0)
+			(hide yes)
+			(show_name no)
+			(do_not_autoplace no)
+			(effects
+				(font
+					(size 1.27 1.27)
+				)
+			)
+		)
+		(pin "1"
+		)
+		(instances
+			(project "Powerboard"
+				(path "/07aca59a-bf87-409f-a974-db5a163ccf8c/c97f42c2-abf8-4b30-857d-14b47bb2334c"
+					(reference "#FLG03")
+					(unit 1)
+				)
+			)
+		)
+	)
+	(symbol
 		(lib_id "SN74HCT245N:SN74HCT245N")
 		(at 120.65 107.95 0)
@@
 			)
 		)
-		(property "Footprint" "N20"
+		(property "Footprint" "SN74HCT245N:N20"
 			(at 120.65 107.95 0)
 			(hide yes)
@@
 		)
 		(property "Description" ""
+			(at 120.65 107.95 0)
+			(hide yes)
+			(show_name no)
+			(do_not_autoplace no)
+			(effects
+				(font
+					(size 1.27 1.27)
+				)
+			)
+		)
+		(property "Untitled Field" ""
 			(at 120.65 107.95 0)
 			(hide yes)
@@
 			)
 		)
-		(property "Footprint" ""
+		(property "Footprint" "Capacitor_SMD:C_0603_1608Metric"
 			(at 96.2152 52.07 0)
 			(hide yes)
@@
 			(at 95.25 48.26 0)
 			(hide yes)
+			(show_name no)
+			(do_not_autoplace no)
+			(effects
+				(font
+					(size 1.27 1.27)
+				)
+			)
+		)
+		(property "Untitled Field" ""
+			(at 95.25 48.26 0)
+			(hide yes)
