File: Powerboard/Motor_Driver.kicad_sch (KiCad schematic)
At the start: 4 parts, among them U5 SN74HCT245N, U6 SN74HCT245N

Commit message: Updated
Parts:
- renumbered C12 to C11, C13 to C12, U5 to U1, U6 to U2
Changed lines of the file:
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@@
 		(dnp no)
 		(fields_autoplaced yes)
-		(property "Reference" "U5"
+		(property "Reference" "U1"
 			(at 146.05 30.48 0)
 			(show_name no)
@@
 			(project "Powerboard"
 				(path "/07aca59a-bf87-409f-a974-db5a163ccf8c/c97f42c2-abf8-4b30-857d-14b47bb2334c"
-					(reference "U5")
+					(reference "U1")
 					(unit 1)
 				)
@@
 		(dnp no)
 		(fields_autoplaced yes)
-		(property "Reference" "#PWR016"
+		(property "Reference" "#PWR015"
 			(at 95.25 77.47 0)
 			(hide yes)
@@
 			(project "Powerboard"
 				(path "/07aca59a-bf87-409f-a974-db5a163ccf8c/c97f42c2-abf8-4b30-857d-14b47bb2334c"
-					(reference "#PWR016")
+					(reference "#PWR015")
 					(unit 1)
 				)
@@
 		(dnp no)
 		(fields_autoplaced yes)
-		(property "Reference" "C13"
+		(property "Reference" "C12"
 			(at 99.06 113.0299 0)
 			(show_name no)
@@
 			(project "Powerboard"
 				(path "/07aca59a-bf87-409f-a974-db5a163ccf8c/c97f42c2-abf8-4b30-857d-14b47bb2334c"
-					(reference "C13")
+					(reference "C12")
 					(unit 1)
 				)
@@
 		(dnp no)
 		(fields_autoplaced yes)
-		(property "Reference" "#PWR014"
+		(property "Reference" "#PWR016"
 			(at 95.25 144.78 0)
 			(hide yes)
@@
 			(project "Powerboard"
 				(path "/07aca59a-bf87-409f-a974-db5a163ccf8c/c97f42c2-abf8-4b30-857d-14b47bb2334c"
-					(reference "#PWR014")
+					(reference "#PWR016")
 					(unit 1)
 				)
@@
 		(dnp no)
 		(fields_autoplaced yes)
-		(property "Reference" "#FLG03"
+		(property "Reference" "#FLG01"
 			(at 93.345 38.1 0)
 			(hide yes)
@@
 			(project "Powerboard"
 				(path "/07aca59a-bf87-409f-a974-db5a163ccf8c/c97f42c2-abf8-4b30-857d-14b47bb2334c"
-					(reference "#FLG03")
+					(reference "#FLG01")
 					(unit 1)
 				)
@@
 		(dnp no)
 		(fields_autoplaced yes)
-		(property "Reference" "U6"
+		(property "Reference" "U2"
 			(at 148.59 97.79 0)
 			(show_name no)
@@
 			(project "Powerboard"
 				(path "/07aca59a-bf87-409f-a974-db5a163ccf8c/c97f42c2-abf8-4b30-857d-14b47bb2334c"
-					(reference "U6")
+					(reference "U2")
 					(unit 1)
 				)
@@
 		(dnp no)
 		(fields_autoplaced yes)
-		(property "Reference" "#PWR027"
+		(property "Reference" "#PWR017"
 			(at 180.34 43.18 0)
 			(hide yes)
@@
 			(project "Powerboard"
 				(path "/07aca59a-bf87-409f-a974-db5a163ccf8c/c97f42c2-abf8-4b30-857d-14b47bb2334c"
-					(reference "#PWR027")
+					(reference "#PWR017")
 					(unit 1)
 				)
@@
 		(dnp no)
 		(fields_autoplaced yes)
-		(property "Reference" "#PWR028"
+		(property "Reference" "#PWR018"
 			(at 182.88 110.49 0)
 			(hide yes)
@@
 			(project "Powerboard"
 				(path "/07aca59a-bf87-409f-a974-db5a163ccf8c/c97f42c2-abf8-4b30-857d-14b47bb2334c"
-					(reference "#PWR028")
+					(reference "#PWR018")
 					(unit 1)
 				)
@@
 		(dnp no)
 		(fields_autoplaced yes)
-		(property "Reference" "C12"
+		(property "Reference" "C11"
 			(at 99.06 46.9899 0)
 			(show_name no)
@@
 			(project "Powerboard"
 				(path "/07aca59a-bf87-409f-a974-db5a163ccf8c/c97f42c2-abf8-4b30-857d-14b47bb2334c"
-					(reference "C12")
+					(reference "C11")
 					(unit 1)
 				)

Commit message: update
Parts:
- removed U1, U2: SN74HCT245N, SN74HCT245N:N20, symbol SN74HCT245N:SN74HCT245N
- added U1, U2: SN74HCT245NSR, SN74HCT245NSR:NS20, symbol SN74HCT245NSR:SN74HCT245NSR
Connections:
- net DIR1_5v: now also U1.12 (B7)
- net DIR2_5v: now also U1.14 (B5)
- net DIR3_5v: now also U1.16 (B3)
- net DIR4_5v: now also U1.18 (B1)
- net DIR5_5v: now also U2.16 (B3)
- net DIR6_5v: now also U2.18 (B1)
- net DIR_1_3v3: now also U1.8 (A7)
- net DIR_2_3v3: now also U1.6 (A5)
- net DIR_3_3v3: now also U1.4 (A3)
- net DIR_4_3v3: now also U1.2 (A1)
- net DIR_5_3v3: now also U2.4 (A3)
- net DIR_6_3v3: now also U2.2 (A1)
- net GND: now also U1.10 (GND), U1.19 (*OE), U2.10 (GND), U2.19 (*OE)
- net PUL1_5V: now also U1.11 (B8)
- net PUL2_5v: now also U1.13 (B6)
- net PUL3_5v: now also U1.15 (B4)
- net PUL4_5v: now also U1.17 (B2)
- net PUL5_5v: now also U2.15 (B4)
- net PUL6_5v: now also U2.17 (B2)
- net PUL_1_3v3: now also U1.9 (A8)
- net PUL_2_3v3: now also U1.7 (A6)
- net PUL_3_3v3: now also U1.5 (A4)
- net PUL_4_3v3: now also U1.3 (A2)
- net PUL_5_3v3: now also U2.5 (A4)
- net PUL_6_3v3: now also U2.3 (A2)
- net Vout_5v: now also U1.1 (DIR), U1.20 (VCC), U2.1 (DIR), U2.20 (VCC)

Commit message: Rev1.1 Done
Finished the board ran DRC all clear
Other:
- company: (none) -> Visionbyte Labs
- title: (none) -> Arm Powerboard
Changed lines of the file:
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@@
 	(generator_version "10.0")
 	(paper "A4")
+	(title_block
+		(title "Arm Powerboard")
+		(date "2026-08-09")
+		(rev "1.1")
+		(company "Visionbyte Labs")
+	)
 	(junction
 		(at 95.25 130.81)

Commit message: Replaced HCT->ACT
Parts:
- removed U1, U2: SN74HCT245NSR, SN74HCT245NSR:NS20, symbol SN74HCT245NSR:SN74HCT245NSR
- added U1, U2: SN74ACT245NSR, SN74ACT245NSR:NS20, symbol SN74ACT245NSR:SN74ACT245NSR
Connections:
- net DIR1_5v: now also U1.12 (B7)
- net DIR2_5v: now also U1.14 (B5)
- net DIR3_5v: now also U1.16 (B3)
- net DIR4_5v: now also U1.18 (B1)
- net DIR5_5v: now also U2.16 (B3)
- net DIR6_5v: now also U2.18 (B1)
- net DIR_1_3v3: now also U1.8 (A7)
- net DIR_2_3v3: now also U1.6 (A5)
- net DIR_3_3v3: now also U1.4 (A3)
- net DIR_4_3v3: now also U1.2 (A1)
- net DIR_5_3v3: now also U2.4 (A3)
- net DIR_6_3v3: now also U2.2 (A1)
- net GND: now also U1.10 (GND), U1.19 (*OE), U2.10 (GND), U2.19 (*OE)
- net PUL1_5V: now also U1.11 (B8)
- net PUL2_5v: now also U1.13 (B6)
- net PUL3_5v: now also U1.15 (B4)
- net PUL4_5v: now also U1.17 (B2)
- net PUL5_5v: now also U2.15 (B4)
- net PUL6_5v: now also U2.17 (B2)
- net PUL_1_3v3: now also U1.9 (A8)
- net PUL_2_3v3: now also U1.7 (A6)
- net PUL_3_3v3: now also U1.5 (A4)
- net PUL_4_3v3: now also U1.3 (A2)
- net PUL_5_3v3: now also U2.5 (A4)
- net PUL_6_3v3: now also U2.3 (A2)
- net Vout_5v: now also U1.1 (DIR), U1.20 (VCC), U2.1 (DIR), U2.20 (VCC)
