File: Powerboard/Powerboard.kicad_pcb (KiCad board)
At the start: 2 copper layers, 5 parts

Commit message: fixed sch
Parts:
- removed REF**: SOT583_MP2338_MNP, MP2338GTL:SOT583_MP2338_MNP-M
- removed REF**: SOIC8E_MPS, MP1584EN:SOIC8E_MPS
- removed REF**: N20, SN74HCT245N:N20
- removed REF**: N20, SN74LVC245AN:N20
- removed REF**: TEENSY41, TEENSY_4.1:TEENSY41
- added C1: 10uF, Capacitor_SMD:C_1206_3216Metric, F.Cu at (179.4, 117.5)
- added C11: 22uF, Capacitor_SMD:C_1206_3216Metric, F.Cu at (113.3, 139.8)
- added C12: 100nF, Capacitor_SMD:C_0603_1608Metric, F.Cu at (191.7, 78.3)
- added C13: 100nF, Capacitor_SMD:C_0603_1608Metric, F.Cu at (191.7, 80.8)
- added C17: 0.1uF, Capacitor_SMD:C_0603_1608Metric, F.Cu at (104.5, 131.3)
- added C18: 22nF, Capacitor_SMD:C_0603_1608Metric, F.Cu at (104.5, 133.8)
- added C19: 0.1uF, Capacitor_SMD:C_0603_1608Metric, F.Cu at (104.5, 136.3)
- added C2: 10uF, Capacitor_SMD:C_1206_3216Metric, F.Cu at (179.4, 120.8)
- added C20: 22uF, Capacitor_SMD:C_1206_3216Metric, F.Cu at (113.3, 143.2)
- added C21: 22uF, Capacitor_SMD:C_0603_1608Metric, F.Cu at (104.5, 138.8)
- added C22: 300pF, Capacitor_SMD:C_0603_1608Metric, F.Cu at (104.5, 141.3)
- added C3: 0.1uF, Capacitor_SMD:C_0603_1608Metric, F.Cu at (170.6, 117.1)
- added C4: 22nF, Capacitor_SMD:C_0603_1608Metric, F.Cu at (170.6, 119.6)
- added C5: 0.1uF, Capacitor_SMD:C_0603_1608Metric, F.Cu at (170.6, 122.1)
- added C6: 22uF, Capacitor_SMD:C_1206_3216Metric, F.Cu at (179.4, 124.2)
- added C7: 22uF, Capacitor_SMD:C_1206_3216Metric, F.Cu at (179.4, 127.5)
- added C8: 470pF, Capacitor_SMD:C_0603_1608Metric, F.Cu at (170.6, 124.6)
- added IC1: TEENSY_4.1, TEENSY_4.1:TEENSY41, F.Cu at (110.4, 64.6)
- added J1: Screw_Terminal_01x02, TerminalBlock_Altech:Altech_AK100_1x02_P5.00mm, F.Cu at (138.1, 97.7)
- added J3: Screw_Terminal_01x12, TerminalBlock_Phoenix:TerminalBlock_Phoenix_MKDS-1,5-12-5.08_1x12_P5.08mm_Horizontal, F.Cu at (106.1, 73.6)
- added J4: Screw_Terminal_01x06, TerminalBlock_Phoenix:TerminalBlock_Phoenix_MKDS-1,5-6_1x06_P5.00mm_Horizontal, F.Cu at (106.0, 97.9)
- added J5: Screw_Terminal_01x06, TerminalBlock_Phoenix:TerminalBlock_Phoenix_MKDS-1,5-6_1x06_P5.00mm_Horizontal, F.Cu at (106.0, 110.0)
- added J6: Screw_Terminal_01x06, TerminalBlock_Phoenix:TerminalBlock_Phoenix_MKDS-1,5-6_1x06_P5.00mm_Horizontal, F.Cu at (106.0, 122.1)
- added J7: Screw_Terminal_01x12, TerminalBlock_Phoenix:TerminalBlock_Phoenix_MKDS-1,5-12-5.08_1x12_P5.08mm_Horizontal, F.Cu at (106.1, 85.7)
- added L1: 6.8uH, Inductor_SMD:L_Bourns_SRP7028A_7.3x6.6mm, F.Cu at (173.5, 111.7)
- added L3: 6.8uH, Inductor_SMD:L_Bourns_SRP7028A_7.3x6.6mm, F.Cu at (115.5, 134.1)
- added R1: 191k, Resistor_SMD:R_0603_1608Metric, F.Cu at (170.6, 127.1)
- added R13: 191k, Resistor_SMD:R_0603_1608Metric, F.Cu at (104.5, 143.8)
- added R14: 49.9k, Resistor_SMD:R_0603_1608Metric, F.Cu at (108.5, 131.3)
- added R15: 10k, Resistor_SMD:R_0603_1608Metric, F.Cu at (108.5, 133.8)
- added R16: 10k, Resistor_SMD:R_0603_1608Metric, F.Cu at (108.5, 136.3)
- added R17: 10k, Resistor_SMD:R_0603_1608Metric, F.Cu at (108.5, 138.8)
- added R18: 90.9k, Resistor_SMD:R_0603_1608Metric, F.Cu at (108.5, 141.3)
- added R2: 49.9k, Resistor_SMD:R_0603_1608Metric, F.Cu at (174.6, 117.1)
- added R3: 100k, Resistor_SMD:R_0603_1608Metric, F.Cu at (174.6, 119.6)
- added R4: 10k, Resistor_SMD:R_0603_1608Metric, F.Cu at (174.6, 122.1)
- added R5: 9.09k, Resistor_SMD:R_0603_1608Metric, F.Cu at (174.6, 124.6)
- added R6: 51k, Resistor_SMD:R_0603_1608Metric, F.Cu at (174.6, 127.1)
- added U1: MP2338GTL-Z, MP2338GTL:SOT583_MP2338_MNP, F.Cu at (180.4, 109.6)
- added U3: MP2338GTL-Z, MP2338GTL:SOT583_MP2338_MNP, F.Cu at (118.1, 140.1)
- added U5: SN74HCT245N, SN74HCT245N:N20, F.Cu at (177.7, 102.8)
- added U6: SN74HCT245N, SN74HCT245N:N20, F.Cu at (188.2, 102.8)
- added U7: SN74LVC245AN, SN74LVC245AN:N20, F.Cu at (177.7, 72.2)
- added U8: SN74LVC245AN, SN74LVC245AN:N20, F.Cu at (188.2, 72.2)
